Commit message: Pure Pursuits Line follower created, process of turning gpsHeading into service

File: src/boost_urdf/robots/boost_stalker.urdf (robot description, URDF)
Before this commit: robot boost_stalker, 28 links, 27 joints
Joints:
- joint front_camera_joint: origin xyz=-0.077693734265045 0.0512582639036014 -1.90500000000204E-05 rpy=3.14159265358979 0.00000015E-12 -2.6117993878 -> xyz=-0.077693734265045 0.0512582639036014 -1.90500000000204E-05 rpy=3.14159265358979 0.0 -2.6117993878

Commit message: Remote push from Duncan #2

File: src/boost_urdf/robots/boost_stalker.urdf (robot description, URDF)
Before this commit: robot boost_stalker, 28 links, 27 joints
Joints:
- joint X-00021: origin xyz=0.0769999999920841 0.115750000014332 0.00200000000075296 -> xyz=0.11 0.115750000014332 0.00200000000075296
